File: SwadgeLEDMatrixTest2.kicad_pcb (KiCad board)
At the start: 2 copper layers, 73.1 x 72.2 mm, 84 parts, among them J1 Conn_01x02_Pin, J2 Conn_01x02_Pin, U1 SAO

Commit message: even now
Parts:
- added REF**: MountingHole_4.3mm_M4_DIN965_Pad, MountingHole:MountingHole_4.3mm_M4_DIN965_Pad, F.Cu at (154.7, 59.6)
- added REF**: MountingHole_4.3mm_M4_DIN965_Pad, MountingHole:MountingHole_4.3mm_M4_DIN965_Pad, F.Cu at (203.1, 71.4)
Other:
- board size 73.1 x 72.2 mm -> 71.3 x 72.2 mm
Changed lines of the file:
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@@
 		)
 	)
+	(footprint "MountingHole:MountingHole_4.3mm_M4_DIN965_Pad"
+		(layer "F.Cu")
+		(at 154.73 59.65)
+		(descr "Mounting Hole 4.3mm, M4, DIN965")
+		(tags "mounting hole 4.3mm m4 din965")
+		(property "Reference" "REF**"
+			(at 0 -4.75 0)
+			(layer "F.SilkS")
+			(hide yes)
+			(effects
+				(font
+					(size 1 1)
+					(thickness 0.15)
+				)
+			)
+		)
+		(property "Value" "MountingHole_4.3mm_M4_DIN965_Pad"
+			(at 0 4.75 0)
+			(layer "F.Fab")
+			(effects
+				(font
+					(size 1 1)
+					(thickness 0.15)
+				)
+			)
+		)
+		(property "Datasheet" ""
+			(at 0 0 0)
+			(unlocked yes)
+			(layer "F.Fab")
+			(hide yes)
+			(effects
+				(font
+					(size 1.27 1.27)
+					(thickness 0.15)
+				)
+			)
+		)
+		(property "Description" ""
+			(at 0 0 0)
+			(unlocked yes)
+			(layer "F.Fab")
+			(hide yes)
+			(effects
+				(font
+					(size 1.27 1.27)
+					(thickness 0.15)
+				)
+			)
+		)
+		(attr exclude_from_pos_files exclude_from_bom)
+		(fp_circle
+			(center 0 0)
+			(end 3.75 0)
+			(stroke
+				(width 0.15)
+				(type solid)
+			)
+			(fill no)
+			(layer "Cmts.User")
+		)
+		(fp_circle
+			(center 0 0)
+			(end 4 0)
+			(stroke
+				(width 0.05)
+				(type solid)
+			)
+			(fill no)
+			(layer "F.CrtYd")
+		)
+		(fp_text user "${REFERENCE}"
+			(at 0 0 0)
+			(layer "F.Fab")
+			(effects
+				(font
+					(size 1 1)
+					(thickness 0.15)
+				)
+			)
+		)
+		(pad "1" thru_hole circle
+			(at 0 0)
+			(size 7.5 7.5)
+			(drill 4.3)
+			(layers "*.Cu" "*.Mask")
+			(remove_unused_layers no)
+		)
+		(embedded_fonts no)
+	)
 	(footprint "LED_SMD:LED_0603_1608Metric_Pad1.05x0.95mm_HandSolder"
 		(layer "F.Cu")
@@
 		)
 	)
+	(footprint "MountingHole:MountingHole_4.3mm_M4_DIN965_Pad"
+		(layer "F.Cu")
+		(at 203.07 71.41)
+		(descr "Mounting Hole 4.3mm, M4, DIN965")
+		(tags "mounting hole 4.3mm m4 din965")
+		(property "Reference" "REF**"
+			(at 0 -4.75 0)
+			(layer "F.SilkS")
+			(hide yes)
+			(effects
+				(font
+					(size 1 1)
+					(thickness 0.15)
+				)
+			)
+		)
+		(property "Value" "MountingHole_4.3mm_M4_DIN965_Pad"
+			(at 0 4.75 0)
+			(layer "F.Fab")
+			(effects
+				(font
+					(size 1 1)
+					(thickness 0.15)
+				)
+			)
+		)
+		(property "Datasheet" ""
+			(at 0 0 0)
+			(unlocked yes)
+			(layer "F.Fab")
+			(hide yes)
+			(effects
+				(font
+					(size 1.27 1.27)
+					(thickness 0.15)
+				)
+			)
+		)
+		(property "Description" ""
+			(at 0 0 0)
+			(unlocked yes)
+			(layer "F.Fab")
+			(hide yes)
+			(effects
+				(font
+					(size 1.27 1.27)
+					(thickness 0.15)
+				)
+			)
+		)
+		(attr exclude_from_pos_files exclude_from_bom)
+		(fp_circle
+			(center 0 0)
+			(end 3.75 0)
+			(stroke
+				(width 0.15)
+				(type solid)
+			)
+			(fill no)
+			(layer "Cmts.User")
+		)
+		(fp_circle
+			(center 0 0)
+			(end 4 0)
+			(stroke
+				(width 0.05)
+				(type solid)
+			)
+			(fill no)
+			(layer "F.CrtYd")
+		)
+		(fp_text user "${REFERENCE}"
+			(at 0 0 0)
+			(layer "F.Fab")
+			(effects
+				(font
+					(size 1 1)
+					(thickness 0.15)
+				)
+			)
+		)
+		(pad "1" thru_hole circle
+			(at 0 0)
+			(size 7.5 7.5)
+			(drill 4.3)
+			(layers "*.Cu" "*.Mask")
+			(remove_unused_layers no)
+		)
+		(embedded_fonts no)
+	)
 	(footprint "Connector_PinHeader_2.54mm:PinHeader_1x02_P2.54mm_Vertical"
 		(layer "F.Cu")
@@
 	)
 	(gr_arc
-		(start 141.05 111.96)
-		(mid 140.349964 111.670036)
-		(end 140.06 110.97)
+		(start 142.8 111.96)
+		(mid 142.099964 111.670036)
+		(end 141.81 110.97)
 		(stroke
 			(width 0.05)
@@
 	)
 	(gr_line
-		(start 140.06 40.73)
-		(end 140.06 110.97)
+		(start 142.8 111.96)
+		(end 212.13 111.96)
 		(stroke
 			(width 0.05)
@@
 	)
 	(gr_line
-		(start 212.13 39.74)
-		(end 141.05 39.74)
+		(start 213.12 110.97)
+		(end 213.12 40.73)
 		(stroke
 			(width 0.05)
@@
 	)
 	(gr_line
-		(start 213.12 110.97)
-		(end 213.12 40.73)
+		(start 141.82 40.73)
+		(end 141.81 110.97)
 		(stroke
 			(width 0.05)
@@
 		(layer "Edge.Cuts")
 	)
-	(gr_arc
-		(start 140.06 40.73)
-		(mid 140.349964 40.029964)
-		(end 141.05 39.74)
+	(gr_line
+		(start 212.13 39.74)
+		(end 142.81 39.74)
 		(stroke
 			(width 0.05)
@@
 	)
 	(gr_arc
-		(start 213.12 110.97)
-		(mid 212.830036 111.670036)
-		(end 212.13 111.96)
+		(start 141.82 40.73)
+		(mid 142.109964 40.029964)
+		(end 142.81 39.74)
 		(stroke
 			(width 0.05)
@@
 		(layer "Edge.Cuts")
 	)
-	(gr_line
-		(start 141.05 111.96)
+	(gr_arc
+		(start 213.12 110.97)
+		(mid 212.830036 111.670036)
 		(end 212.13 111.96)
 		(stroke
@@
 		(layer "B.SilkS")
 		(pts
-			(xy 145.1 39.8) (xy 145.31 111.9)
+			(xy 213.19 86.42) (xy 141.92 87.32)
 		)
-		(height -0.73)
-		(orientation 1)
+		(height 0.78)
+		(orientation 0)
 		(format
 			(prefix "")
@@
 			(keep_text_aligned yes)
 		)
-		(gr_text "72.1"
-			(at 143.27 75.85 90)
+		(gr_text "71.27"
+			(at 177.555 86.1 0)
 			(layer "B.SilkS")
 			(effects
@@
 		(layer "B.SilkS")
 		(pts
-			(xy 212.82 69.33) (xy 140.09 71.1)
+			(xy 144.56 111.96) (xy 145.02 39.74)
 		)
-		(height -3.55)
-		(orientation 0)
+		(height 0.4)
+		(orientation 1)
 		(format
 			(prefix "")
@@
 			(keep_text_aligned yes)
 		)
-		(gr_text "72.73"
-			(at 176.455 64.68 0)
+		(gr_text "72.22"
+			(at 143.86 75.85 90)
 			(layer "B.SilkS")
 			(effects
